File: RF.kicad_sch (KiCad schematic)
At the start: 27 parts, among them J1 Conn_Coaxial, SW1 SW_DIP_x01, U1 AD8307, U2 L7805

Commit message: C11 przeniesiony
Connections:
- net VCC: now also C11.1
- net V_BAT: no longer C11.1
Other:
- moved on the sheet: C11
Changed lines of the file:
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@@
-	)
-	(junction
-		(at 264.16 34.29)
-		(diameter 0)
-		(color 0 0 0 0)
 	)
 	(junction
@@
 	(wire
 		(pts
-			(xy 267.97 34.29) (xy 264.16 34.29)
+			(xy 262.89 34.29) (xy 267.97 34.29)
 		)
 		(stroke
@@
 	(wire
 		(pts
-			(xy 264.16 34.29) (xy 262.89 34.29)
-		)
-		(stroke
-			(width 0)
-			(type default)
-		)
-	)
-	(wire
-		(pts
 			(xy 208.28 102.87) (xy 214.63 102.87)
 		)
@@
 	(wire
 		(pts
-			(xy 264.16 34.29) (xy 264.16 36.83)
-		)
-		(stroke
-			(width 0)
-			(type default)
-		)
-	)
-	(wire
-		(pts
 			(xy 87.63 91.44) (xy 92.71 91.44)
 		)
@@
 	(wire
 		(pts
+			(xy 196.85 34.29) (xy 196.85 36.83)
+		)
+		(stroke
+			(width 0)
+			(type default)
+		)
+	)
+	(wire
+		(pts
 			(xy 92.71 82.55) (xy 92.71 91.44)
 		)
@@
 	(wire
 		(pts
-			(xy 264.16 44.45) (xy 264.16 50.8)
+			(xy 196.85 44.45) (xy 196.85 50.8)
 		)
 		(stroke
@@
 		(pts
 			(xy 173.99 100.33) (xy 184.15 100.33)
+		)
+		(stroke
+			(width 0)
+			(type default)
+		)
+	)
+	(wire
+		(pts
+			(xy 212.09 34.29) (xy 196.85 34.29)
 		)
 		(stroke
@@
 	(symbol
 		(lib_id "power:GNDPWR")
-		(at 264.16 50.8 0)
+		(at 196.85 50.8 0)
 		(unit 1)
 		(exclude_from_sim no)
@@
 		(fields_autoplaced yes)
 		(property "Reference" "#PWR012"
-			(at 264.16 55.88 0)
+			(at 196.85 55.88 0)
 			(effects
 				(font
@@
 		)
 		(property "Value" "GNDPWR"
-			(at 264.033 54.61 0)
+			(at 196.723 54.61 0)
 			(effects
 				(font
@@
 		)
 		(property "Footprint" ""
-			(at 264.16 52.07 0)
+			(at 196.85 52.07 0)
 			(effects
 				(font
@@
 		)
 		(property "Datasheet" ""
-			(at 264.16 52.07 0)
+			(at 196.85 52.07 0)
 			(effects
 				(font
@@
 		)
 		(property "Description" "Power symbol creates a global label with name \"GNDPWR\" , global ground"
-			(at 264.16 50.8 0)
+			(at 196.85 50.8 0)
 			(effects
 				(font
@@
 	(symbol
 		(lib_id "Device:C_Polarized_US")
-		(at 264.16 40.64 0)
+		(at 196.85 40.64 0)
 		(unit 1)
 		(exclude_from_sim no)
@@
 		(fields_autoplaced yes)
 		(property "Reference" "C11"
-			(at 267.97 38.7349 0)
+			(at 200.66 38.7349 0)
 			(effects
 				(font
@@
 		)
 		(property "Value" "10u"
-			(at 267.97 41.2749 0)
+			(at 200.66 41.2749 0)
 			(effects
 				(font
@@
 		)
 		(property "Footprint" "Capacitor_SMD:CP_Elec_6.3x5.3"
-			(at 264.16 40.64 0)
+			(at 196.85 40.64 0)
 			(effects
 				(font
@@
 		)
 		(property "Datasheet" "~"
-			(at 264.16 40.64 0)
+			(at 196.85 40.64 0)
 			(effects
 				(font
@@
 		)
 		(property "Description" "Polarized capacitor, US symbol"
-			(at 264.16 40.64 0)
-			(effects
-				(font
+			(at 196.85 40.64 0)
+			(effects
+				(font

Commit message: ostatnie zmiany 09.08.2024
Changed lines of the file:
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@@
 	)
 	(junction
+		(at 148.59 38.1)
+		(diameter 0)
+		(color 0 0 0 0)
+	)
+	(junction
 		(at 232.41 34.29)
 		(diameter 0)
@@
 	(wire
 		(pts
+			(xy 148.59 38.1) (xy 156.21 38.1)
+		)
+		(stroke
+			(width 0)
+			(type default)
+		)
+	)
+	(wire
+		(pts
 			(xy 92.71 106.68) (xy 92.71 109.22)
 		)
@@
 	(wire
 		(pts
-			(xy 143.51 38.1) (xy 156.21 38.1)
+			(xy 143.51 38.1) (xy 148.59 38.1)
 		)
 		(stroke
@@
 					(unit 1)
 				)
+			)
+		)
+	)
+	(symbol
+		(lib_id "power:PWR_FLAG")
+		(at 148.59 38.1 0)
+		(unit 1)
+		(exclude_from_sim no)
+		(in_bom yes)
+		(on_board yes)
+		(dnp no)
+		(fields_autoplaced yes)
+		(property "Reference" "#FLG01"
+			(at 148.59 36.195 0)
+			(effects
+				(font
+					(size 1.27 1.27)
+				)
+				(hide yes)
+			)
+		)
+		(property "Value" "PWR_FLAG"
+			(at 148.59 33.02 0)
+			(effects
+				(font
+					(size 1.27 1.27)
+				)
+			)
+		)
+		(property "Footprint" ""
+			(at 148.59 38.1 0)
+			(effects
+				(font
+					(size 1.27 1.27)
+				)
+				(hide yes)
+			)
+		)
+		(property "Datasheet" "~"
+			(at 148.59 38.1 0)
+			(effects
+				(font
+					(size 1.27 1.27)
+				)
+				(hide yes)
+			)
+		)
+		(property "Description" "Special symbol for telling ERC where power comes from"
+			(at 148.59 38.1 0)
+			(effects
+				(font
+					(size 1.27 1.27)
+				)
+				(hide yes)
+			)
+		)
+		(pin "1"
+		)
+		(instances
+			(project ""
+				(path "/6e9b0ecb-5ff8-4cea-bb01-e8c92e636c95/09627191-d48d-42a8-a392-355888bdeeaa"
+					(reference "#FLG01")
+					(unit 1)
+				)

Commit message: usunięte część ostrzeżeń i błędów
Connections:
- net VCC: now also U2.3 (OUT); no longer U2.1 (OUT)
- net at C7.1, R5.1: now also U2.1 (IN); no longer U2.3 (IN)
Changed lines of the file:
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@@
 		)
 		(property "Footprint" "Package_TO_SOT_SMD:SOT-89-3_Handsoldering"
-			(at 221.615 30.48 0)
+			(at 223.012 14.986 0)
 			(effects
 				(font
@@
 		)
 		(property "Datasheet" "http://www.st.com/content/ccc/resource/technical/document/datasheet/41/4f/b3/b0/12/d4/47/88/CD00000444.pdf/files/CD00000444.pdf/jcr:content/translations/en.CD00000444.pdf"
-			(at 222.25 33.02 0)
+			(at 221.488 12.446 0)
 			(effects
 				(font
@@
 		)
 		(property "Description" "Positive 1.5A 35V Linear Regulator, Fixed Output 5V, TO-220/TO-263/TO-252"
-			(at 222.25 34.29 0)
+			(at 225.298 13.462 0)
 			(effects
 				(font
