File: projekt.kicad_pcb (KiCad board)
At the start: 2 copper layers, 90 x 35 mm, 38 parts, among them J1 Conn_Coaxial, J2 OLED, SW1 SW_DIP_x01, U1 AD8307, U2 L7805

Commit message: poprawione piny RP2040 na płytce
Routing:
- net Net-(RP2040-zero1-GP13): track 6.06 -> 20.5 mm
- net /uC/RST: track 16.4 -> 12.8 mm
- net Net-(RP2040-zero1-GP11): track 6.22 -> 7.52 mm
- net Net-(RP2040-zero1-GP10): track 3.47 -> 4.61 mm
- net /uC/3V3: track 52.1 -> 52.9 mm
Changed lines of the file:
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@@
 		)
 		(pad "10" thru_hole circle
-			(at 1.38 -1.59 180)
+			(at 14.08 -1.38 180)
 			(size 1.8 1.8)
 			(drill 1)
@@
 		)
 		(pad "11" thru_hole circle
-			(at 14.08 -1.38 180)
+			(at 11.54 -1.38 180)
 			(size 1.8 1.8)
 			(drill 1)
@@
 		)
 		(pad "12" thru_hole circle
-			(at 11.54 -1.38 180)
+			(at 9 -1.38 180)
 			(size 1.8 1.8)
 			(drill 1)
@@
 		)
 		(pad "13" thru_hole circle
-			(at 9 -1.38 180)
+			(at 6.46 -1.38 180)
 			(size 1.8 1.8)
 			(drill 1)
@@
 		)
 		(pad "14" thru_hole circle
-			(at 6.46 -1.38 180)
+			(at 3.92 -1.38 180)
 			(size 1.8 1.8)
 			(drill 1)
@@
 		)
 		(pad "15" thru_hole circle
-			(at 3.92 -1.38 180)
+			(at 1.38 -1.59 180)
 			(size 1.8 1.8)
 			(drill 1)
@@
 	)
 	(segment
-		(start 82.143 29.083)
-		(end 82.313 29.253)
-		(width 0.2)
+		(start 84.853 32.241)
+		(end 84.836 32.258)
+		(width 0.2032)
 		(layer "F.Cu")
 		(net 14)
 	)
 	(segment
-		(start 82.143 32.071)
-		(end 82.313 32.241)
-		(width 0.2032)
+		(start 82.143 29.643)
+		(end 82.143 29.083)
+		(width 0.2)
 		(layer "F.Cu")
 		(net 14)
@@
 	(segment
 		(start 82.143 29.083)
-		(end 82.143 32.071)
-		(width 0.2032)
+		(end 82.313 29.253)
+		(width 0.2)
 		(layer "F.Cu")
 		(net 14)
 	)
 	(segment
-		(start 91.824 33.721)
-		(end 89.467 33.721)
+		(start 84.853 32.241)
+		(end 84.741 32.241)
 		(width 0.2)
 		(layer "F.Cu")
-		(net 15)
+		(net 14)
 	)
 	(segment
-		(start 85.9487 29.083)
-		(end 85.243 29.083)
+		(start 84.741 32.241)
+		(end 82.143 29.643)
 		(width 0.2)
 		(layer "F.Cu")
-		(net 15)
+		(net 14)
 	)
 	(segment
-		(start 88.6631 31.7974)
-		(end 85.9487 29.083)
+		(start 92.5 33.320943)
+		(end 88.262057 29.083)
 		(width 0.2)
 		(layer "F.Cu")
@@
 	)
 	(segment
-		(start 94.452 36.349)
-		(end 91.824 33.721)
+		(start 92.5 34.397)
+		(end 92.5 33.320943)
 		(width 0.2)
 		(layer "F.Cu")
@@
 	)
 	(segment
-		(start 88.6631 32.9171)
-		(end 88.6631 31.7974)
+		(start 94.452 36.349)
+		(end 92.5 34.397)
 		(width 0.2)
 		(layer "F.Cu")
@@
 	)
 	(segment
-		(start 89.467 33.721)
-		(end 88.6631 32.9171)
+		(start 88.262057 29.083)
+		(end 85.243 29.083)
 		(width 0.2)
 		(layer "F.Cu")
@@
 	)
 	(segment
-		(start 91.8924 36.3294)
+		(start 83.693 29.342744)
+		(end 85.391256 31.041)
+		(width 0.2)
+		(layer "F.Cu")
+		(net 18)
+	)
+	(segment
+		(start 88.733 31.883943)
+		(end 88.733 32.948057)
+		(width 0.2)
+		(layer "F.Cu")
+		(net 18)
+	)
+	(segment
+		(start 90.430057 33.791)
+		(end 92.5 35.860943)
+		(width 0.2)
+		(layer "F.Cu")
+		(net 18)
+	)
+	(segment
+		(start 87.890057 31.041)
+		(end 88.733 31.883943)
+		(width 0.2)
+		(layer "F.Cu")
+		(net 18)
+	)
+	(segment
+		(start 92.5 36.937)
 		(end 94.452 38.889)
+		(width 0.2)
+		(layer "F.Cu")
+		(net 18)
+	)
+	(segment
+		(start 83.693 29)
+		(end 83.693 29.342744)
+		(width 0.2)
+		(layer "F.Cu")
+		(net 18)
+	)
+	(segment
+		(start 92.5 35.860943)
+		(end 92.5 36.937)
+		(width 0.2)
+		(layer "F.Cu")
+		(net 18)
+	)
+	(segment
+		(start 89.575943 33.791)
+		(end 90.430057 33.791)
+		(width 0.2)
+		(layer "F.Cu")
+		(net 18)
+	)
+	(segment
+		(start 83.693 29)
+		(end 83.693 29.345008)
 		(width 0.2032)
 		(layer "F.Cu")
@@
 	(segment
 		(start 83.693 26.898)
-		(end 83.693 29.38168)
+		(end 83.693 29)
 		(width 0.2032)
 		(layer "F.Cu")
@@
 	)
 	(segment
-		(start 86.0546 34.0546)
-		(end 88.3294 36.3294)
-		(width 0.2032)
+		(start 85.391256 31.041)
+		(end 87.890057 31.041)
+		(width 0.2)
 		(layer "F.Cu")
 		(net 18)
@@
 	)
 	(segment
-		(start 86.0546 31.74328)
-		(end 86.0546 34.0546)
-		(width 0.2032)
+		(start 88.733 32.948057)
+		(end 89.575943 33.791)
+		(width 0.2)
 		(layer "F.Cu")
 		(net 18)
 	)
 	(segment
-		(start 83.693 29.38168)
-		(end 86.0546 31.74328)
+		(start 77.5 23.5)
+		(end 72 29)
 		(width 0.2032)
 		(layer "F.Cu")
-		(net 18)
+		(net 19)
 	)
 	(segment
-		(start 88.3294 36.3294)
-		(end 91.8924 36.3294)
+		(start 92 31.357)
+		(end 94.452 33.809)
 		(width 0.2032)
 		(layer "F.Cu")
-		(net 18)
+		(net 19)
 	)
 	(segment
-		(start 92 26)
-		(end 92 31.357)
+		(start 82 23.5)
+		(end 77.5 23.5)
 		(width 0.2032)
 		(layer "F.Cu")
@@
 	)
 	(segment
-		(start 72 29)
-		(end 76.5 24.5)
-		(width 0.2032)
+		(start 84.5 23.5)
+		(end 82 23.5)
+		(width 0.2)
 		(layer "F.Cu")
 		(net 19)
 	)
 	(segment
-		(start 92 31.357)
-		(end 94.452 33.809)
+		(start 92 26)
+		(end 92 31.357)
 		(width 0.2032)
 		(layer "F.Cu")
@@
 	)
 	(segment
-		(start 90.5 24.5)
+		(start 89.5 23.5)
 		(end 92 26)
 		(width 0.2032)
@@
 	)
 	(segment
-		(start 73.191 47.691)
-		(end 72 46.5)
+		(start 84.5 23.5)
+		(end 89.5 23.5)
 		(width 0.2032)
 		(layer "F.Cu")
@@
 	)
 	(segment
-		(start 72 43)
-		(end 72 29)
+		(start 73.191 47.691)
+		(end 72 46.5)
 		(width 0.2032)
 		(layer "F.Cu")
@@
 	)
 	(segment
-		(start 76.5 24.5)
-		(end 90.5 24.5)
+		(start 72 29)
+		(end 72 43)
 		(width 0.2032)
 		(layer "F.Cu")
@@
 	)
 	(segment
-		(start 84.836 37.336)
-		(end 86.3694 38.8694)
-		(width 0.2032)
+		(start 87.393 34.148057)
+		(end 89.435943 36.191)
+		(width 0.2)
 		(layer "F.Cu")
 		(net 20)
 	)
 	(segment
-		(start 84.836 32.258)
-		(end 84.836 37.336)
-		(width 0.2032)
+		(start 87.393 32.241)
+		(end 87.393 34.148057)
+		(width 0.2)
 		(layer "F.Cu")
 		(net 20)
 	)
 	(segment
-		(start 84.853 32.241)
-		(end 84.836 32.258)
-		(width 0.2032)
+		(start 90.691 36.191)
+		(end 91.8924 37.3924)
+		(width 0.2)
 		(layer "F.Cu")
 		(net 20)
 	)
 	(segment
-		(start 86.3694 38.8694)
+		(start 91.8924 37.3924)
 		(end 91.8924 38.8694)
-		(width 0.2032)
+		(width 0.2)
+		(layer "F.Cu")
+		(net 20)
+	)
+	(segment
+		(start 89.435943 36.191)
+		(end 90.691 36.191)
+		(width 0.2)
 		(layer "F.Cu")
 		(net 20)
@@
 	)
 	(segment
-		(start 79.73 26.035)
-		(end 79.73 32.198)
-		(width 0.2032)
+		(start 79.73 29.658)
+		(end 79.73 26.035)
+		(width 0.2)
 		(layer "F.Cu")
 		(net 25)
 	)
 	(segment
-		(start 79.73 32.198)
-		(end 79.773 32.241)
+		(start 82.313 32.241)
+		(end 79.73 29.658)
+		(width 0.2)
+		(layer "F.Cu")
+		(net 25)
+	)
+	(segment
+		(start 82.143 32.071)
+		(end 82.313 32.241)
 		(width 0.2032)
 		(layer "F.Cu")
@@
 	)
 	(segment
+		(start 79.73 32.198)
+		(end 79.773 32.241)
+		(width 0.2032)
+		(layer "F.Cu")
+		(net 28)
+	)
+	(segment
+		(start 90.017 32.367)
+		(end 89.933 32.451)
+		(width 0.2)
+		(layer "F.Cu")
+		(net 32)
+	)
+	(segment
 		(start 32.5485 44.574)
 		(end 32.6755 44.447)
@@
 	)
 	(segment
-		(start 89.933 32.451)
-		(end 89.933 26.627)
-		(width 0.2032)
+		(start 87 24.5)
+		(end 89.043 26.543)
+		(width 0.2)
 		(layer "F.Cu")
 		(net 42)
 	)
 	(segment
-		(start 90.017 32.367)
-		(end 89.933 32.451)
+		(start 79 24.5)
+		(end 87 24.5)
+		(width 0.2)
+		(layer "F.Cu")
+		(net 42)
+	)
+	(segment
+		(start 77.233 32.241)
+		(end 77.233 26.267)
+		(width 0.2)
+		(layer "F.Cu")
+		(net 42)
+	)
+	(segment
+		(start 89.043 26.543)
+		(end 90.017 26.543)
+		(width 0.2)
+		(layer "F.Cu")
+		(net 42)
+	)
+	(segment
+		(start 77.233 26.267)
+		(end 79 24.5)
 		(width 0.2)
 		(layer "F.Cu")
